File: AVIONICS/AVIONICS-PCB/Avionics_PCB/Avionics_PCB.kicad_pcb (KiCad board)
At the start: 2 copper layers, 27 parts, among them J1 U-Blox M8N, J2 MPU9250, J3 Micro_SD_Card_Det1, J4 DS1302, J5 USB_B_Micro, J6 Bat_Conn, SW1 EN_SW, SW2 IO0_SW, U1 ESP32-S3-WROOM-1, U2 LoRa_RA-02, U3 BMP280, U4 ME6211C33M5

Commit message: pcb dev
Parts:
- J3: footprint Connector_Card:microSD_HC_Hirose_DM3D-SF -> Connector_Card:microSD_HC_Hirose_DM3AT-SF-PEJM5
- moved R3 83.1 mm to (100.5, 131.2), turned to 180 degrees
- moved J4 80.9 mm to (122.5, 141.3), turned to -90 degrees
- moved R4 79.6 mm to (100.5, 129.2), turned to 180 degrees
- moved J2 74.0 mm to (104.8, 125.8), turned to 90 degrees
- moved R1 66.0 mm to (95.0, 83.2)
- moved U3 65.1 mm to (97.1, 131.6)
- moved C6 60.0 mm to (94.5, 131.2), turned to 90 degrees
- moved C7 59.2 mm to (95.2, 134.0)
- moved C4 58.7 mm to (104.0, 75.9), turned to -90 degrees
- moved C5 58.5 mm to (103.5, 79.7), turned to 90 degrees
- moved J1 57.0 mm to (131.5, 161.3)
- moved C3 55.2 mm to (105.9, 75.9), turned to -90 degrees
- moved C9 52.6 mm to (97.4, 119.7)
- moved C10 52.5 mm to (97.5, 121.7)
- moved R5 52.2 mm to (118.6, 111.3), turned to 180 degrees
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Connections:
- C1 pad 1: AD0 -> GND
- C10 pad 1: 3V3 -> GND
- C10 pad 2: Net-(U2-VDD) -> 3V3
- C2 pad 2: AD0 -> GND
- C3 pad 1: 3V3 -> GND
- C3 pad 2: Net-(U1-3V3) -> 3V3
- C4 pad 1: 3V3 -> GND
- C4 pad 2: Net-(U1-3V3) -> 3V3
- C5 pad 2: AD0 -> GND
- C6 pad 2: AD0 -> GND
- C7 pad 2: AD0 -> GND
- C8 pad 1: AD0 -> GND
- C9 pad 1: 3V3 -> GND
- C9 pad 2: Net-(U2-VDD) -> 3V3
- J1 pad 1: AD0 -> GND
- J1 pad 3: GPS_TX -> GPS_RX
- J2 pad 2: AD0 -> GND
- J2 pad 7: AD0 -> GND
- J3 pad 10: AD0 -> GND
- J3 pad 6: AD0 -> GND
- J4 pad 3: AD0 -> GND
- J5 pad 5: AD0 -> GND
- J5 pad 6: AD0 -> GND
- J6 pad 2: AD0 -> GND
- SW1 pad 1: AD0 -> GND
- SW2 pad 1: AD0 -> GND
- U1 pad 1: AD0 -> GND
- U1 pad 2: Net-(U1-3V3) -> 3V3
- U1 pad 40: AD0 -> GND
- U1 pad 41: AD0 -> GND
- U2 pad 1: AD0 -> GND
- U2 pad 16: AD0 -> GND
- U2 pad 2: AD0 -> GND
- U2 pad 3: Net-(U2-VDD) -> 3V3
- U2 pad 9: AD0 -> GND
- U3 pad 1: AD0 -> GND
- U3 pad 5: AD0 -> GND
- U3 pad 7: AD0 -> GND
- U4 pad 2: AD0 -> GND
Routing:
- net 3V3: track 0.00 -> 200.2 mm, vias 0 -> 8
- net GND: track 0.00 -> 132.2 mm, vias 0 -> 4
- net GPS_RX: track 0.00 -> 97.0 mm, vias 0 -> 1
- net GPS_TX: track 0.00 -> 94.9 mm, vias 0 -> 1
- net RTC_SCLK: track 0.00 -> 78.8 mm, vias 0 -> 2
- net RTC_RST: track 0.00 -> 71.9 mm, vias 0 -> 3
- net RTC_IO: track 0.00 -> 64.5 mm, vias 0 -> 1
- net SDA: track 0.00 -> 62.4 mm, vias 0 -> 2
- net LORA_DIO0: track 0.00 -> 56.9 mm, vias 0 -> 2
- net SPI_MISO: track 0.00 -> 55.7 mm, vias 0 -> 4
- net SPI_MOSI: track 0.00 -> 50.4 mm, vias 0 -> 2
- net SCL: track 0.00 -> 50.3 mm, vias 0 -> 2
- net SPI_SCK: track 0.00 -> 47.7 mm, vias 0 -> 2
- net D-: track 0.00 -> 38.8 mm, vias 0 -> 2
- net LORA_RST: track 0.00 -> 38.3 mm
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- added copper zone on In1.Cu, net GND
Other:
- board outline added: 46.7 x 109.2 mm
- copper layers 2 -> 4

Commit message: Avionics CAD progression
Parts:
- added G***: LOGO, LOGO, B.Cu at (116.0, 153.0)
- added REF**: MountingHole_3.2mm_M3, MountingHole:MountingHole_3.2mm_M3, F.Cu at (96.0, 143.5)
- added REF**: MountingHole_3.2mm_M3, MountingHole:MountingHole_3.2mm_M3, F.Cu at (96.0, 178.5)
- added REF**: MountingHole_3.2mm_M3, MountingHole:MountingHole_3.2mm_M3, F.Cu at (96.0, 90.5)
- added REF**: MountingHole_3.2mm_M3, MountingHole:MountingHole_3.2mm_M3, F.Cu at (135.0, 178.5)
- added REF**: MountingHole_3.2mm_M3, MountingHole:MountingHole_3.2mm_M3, F.Cu at (135.0, 143.5)
- J3: value Micro_SD_Card_Det1 -> Micro_SD_card
- U2: value LoRa_RA-02 -> LoRa_Ra-02
- moved J6 1.00 mm to (133.5, 90.5), turned to 0 degrees
Routing:
- net GPS_RX: track 97.0 -> 91.8 mm
- net GPS_TX: track 94.9 -> 90.4 mm
- net 3V3: track 200.2 -> 196.0 mm
- net SCL: track 50.3 -> 53.2 mm
- net GND: track 132.2 -> 130.4 mm
- net SDA: track 62.4 -> 64.1 mm
- net SPI_SCK: track 47.7 -> 48.4 mm
- net LORA_CS: track 26.5 -> 27.1 mm
Other:
- board size 46.7 x 109.2 mm -> 47.8 x 109.2 mm
- board text added: "BAT_Conn"
- board text added: "Designed By Parth Dhiman October,2026"
