File: AVIONICS/AVIONICS-PCB/Avionics_PCB/Avionics_PCB.kicad_sch (KiCad schematic)
At the start: 27 parts, among them J1 U-Blox M8N, J2 MPU9250, J3 Micro_SD_Card_Det1, J4 DS1302, J5 USB_B_Micro, J6 Bat_Conn, SW1 EN_SW, SW2 IO0_SW, U1 ESP32-S3-WROOM-1, U2 LoRa_RA-02, U3 BMP280, U4 ME6211C33M5

Commit message: pcb dev
Parts:
- J3: footprint Connector_Card:microSD_HC_Hirose_DM3D-SF -> Connector_Card:microSD_HC_Hirose_DM3AT-SF-PEJM5
Connections:
- net 3V3: now also C10.2, C3.2, C4.2, C9.2, U1.2 (3V3), U2.3 (VDD); no longer C10.1, C3.1, C4.1, C9.1
- net GND: now also C10.1, C3.1, C4.1, C9.1
- net GPS_RX: now also J1.3 (Pin_3)
- net GPS_TX: no longer J1.3 (Pin_3)
Changed lines of the file:
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@@
 	)
 	(junction
-		(at 140.97 104.14)
+		(at 36.83 97.79)
 		(diameter 0)
 		(color 0 0 0 0)
 	)
 	(junction
-		(at 135.89 38.1)
+		(at 54.61 90.17)
 		(diameter 0)
 		(color 0 0 0 0)
 	)
 	(junction
-		(at 36.83 97.79)
+		(at 57.15 85.09)
 		(diameter 0)
 		(color 0 0 0 0)
 	)
 	(junction
-		(at 54.61 90.17)
+		(at 144.78 124.46)
 		(diameter 0)
 		(color 0 0 0 0)
 	)
 	(junction
-		(at 57.15 85.09)
+		(at 31.75 184.15)
 		(diameter 0)
 		(color 0 0 0 0)
 	)
 	(junction
-		(at 31.75 184.15)
+		(at 140.97 46.99)
 		(diameter 0)
 		(color 0 0 0 0)
@@
 	)
 	(junction
-		(at 134.62 116.84)
-		(diameter 0)
-		(color 0 0 0 0)
-	)
-	(junction
 		(at 220.98 39.37)
 		(diameter 0)
@@
 	)
 	(junction
+		(at 140.97 38.1)
+		(diameter 0)
+		(color 0 0 0 0)
+	)
+	(junction
 		(at 220.98 49.53)
 		(diameter 0)
@@
 	(wire
 		(pts
-			(xy 132.08 38.1) (xy 135.89 38.1)
+			(xy 25.4 173.99) (xy 25.4 171.45)
 		)
 		(stroke
@@
 	(wire
 		(pts
-			(xy 25.4 173.99) (xy 25.4 171.45)
+			(xy 87.63 168.91) (xy 92.71 168.91)
 		)
 		(stroke
@@
 	(wire
 		(pts
-			(xy 87.63 168.91) (xy 92.71 168.91)
+			(xy 140.97 38.1) (xy 146.05 38.1)
 		)
 		(stroke
@@
 	(wire
 		(pts
-			(xy 140.97 104.14) (xy 140.97 102.87)
+			(xy 137.16 46.99) (xy 140.97 46.99)
 		)
 		(stroke
@@
 	(wire
 		(pts
-			(xy 135.89 38.1) (xy 146.05 38.1)
-		)
-		(stroke
-			(width 0)
-			(type default)
-		)
-	)
-	(wire
-		(pts
-			(xy 132.08 115.57) (xy 134.62 115.57)
+			(xy 135.89 38.1) (xy 140.97 38.1)
 		)
 		(stroke
@@
 	(wire
 		(pts
-			(xy 138.43 104.14) (xy 140.97 104.14)
-		)
-		(stroke
-			(width 0)
-			(type default)
-		)
-	)
-	(wire
-		(pts
 			(xy 229.87 60.96) (xy 251.46 60.96)
 		)
@@
 	(wire
 		(pts
-			(xy 134.62 115.57) (xy 134.62 116.84)
-		)
-		(stroke
-			(width 0)
-			(type default)
-		)
-	)
-	(wire
-		(pts
 			(xy 80.01 34.29) (xy 76.2 34.29)
 		)
@@
 	(wire
 		(pts
-			(xy 140.97 106.68) (xy 140.97 104.14)
+			(xy 259.08 29.21) (xy 259.08 38.1)
 		)
 		(stroke
@@
 	(wire
 		(pts
-			(xy 259.08 29.21) (xy 259.08 38.1)
+			(xy 25.4 171.45) (xy 31.75 171.45)
 		)
 		(stroke
@@
 	(wire
 		(pts
-			(xy 25.4 171.45) (xy 31.75 171.45)
+			(xy 220.98 52.07) (xy 218.44 52.07)
 		)
 		(stroke
@@
 	(wire
 		(pts
-			(xy 220.98 52.07) (xy 218.44 52.07)
+			(xy 85.09 41.91) (xy 80.01 41.91)
 		)
 		(stroke
@@
 	(wire
 		(pts
-			(xy 85.09 41.91) (xy 80.01 41.91)
+			(xy 199.39 52.07) (xy 200.66 52.07)
 		)
 		(stroke
@@
 	(wire
 		(pts
-			(xy 199.39 52.07) (xy 200.66 52.07)
+			(xy 149.86 124.46) (xy 144.78 124.46)
 		)
 		(stroke
@@
 		)
 	)
+	(global_label "GND"
+		(shape input)
+		(at 240.03 91.44 180)
+		(fields_autoplaced yes)
+		(effects
+			(font
+				(size 1.27 1.27)
+			)
+			(justify right)
+		)
+		(property "Intersheetrefs" "${INTERSHEET_REFS}"
+			(at 233.1743 91.44 0)
+			(effects
+				(font
+					(size 1.27 1.27)
+				)
+				(justify right)
+				(hide yes)
+			)
+		)
+	)
 	(global_label "RTC_SCLK"
 		(shape input)
@@
 		)
 	)
+	(global_label "3V3"
+		(shape input)
+		(at 149.86 124.46 0)
+		(fields_autoplaced yes)
+		(effects
+			(font
+				(size 1.27 1.27)
+			)
+			(justify left)
+		)
+		(property "Intersheetrefs" "${INTERSHEET_REFS}"
+			(at 156.3528 124.46 0)
+			(effects
+				(font
+					(size 1.27 1.27)
+				)
+				(justify left)
+				(hide yes)
+			)
+		)
+	)
 	(global_label "GPS_TX"
 		(shape input)
@@
 		)
 	)
+	(global_label "GND"
+		(shape input)
+		(at 139.7 116.84 90)
+		(fields_autoplaced yes)
+		(effects
+			(font
+				(size 1.27 1.27)
+			)
+			(justify left)
+		)
+		(property "Intersheetrefs" "${INTERSHEET_REFS}"
+			(at 139.7 109.9843 90)
+			(effects
+				(font
+					(size 1.27 1.27)
+				)
+				(justify left)
+				(hide yes)
+			)
+		)
+	)
 	(global_label "SPI_MOSI"
 		(shape input)
@@
 		)
 	)
-	(global_label "GPS_TX"
+	(global_label "GPS_RX"
 		(shape input)
 		(at 238.76 138.43 180)
@@
 		)
 		(property "Intersheetrefs" "${INTERSHEET_REFS}"
-			(at 228.8806 138.43 0)
+			(at 228.5782 138.43 0)
 			(effects
 				(font
@@
 		)
 	)
-	(global_label "3V3"
-		(shape input)
-		(at 132.08 115.57 180)
-		(fields_autoplaced yes)
-		(effects
-			(font
-				(size 1.27 1.27)
-			)
-			(justify right)
-		)
-		(property "Intersheetrefs" "${INTERSHEET_REFS}"
-			(at 125.5872 115.57 0)
-			(effects
-				(font
-					(size 1.27 1.27)
-				)
-				(justify right)
-				(hide yes)
-			)
-		)
-	)
-	(global_label "AD0"
-		(shape input)
-		(at 138.43 104.14 180)
-		(fields_autoplaced yes)
-		(effects
-			(font
-				(size 1.27 1.27)
-			)
-			(justify right)
-		)
-		(property "Intersheetrefs" "${INTERSHEET_REFS}"
-			(at 131.8767 104.14 0)
-			(effects
-				(font
-					(size 1.27 1.27)
-				)
-				(justify right)
-				(hide yes)
-			)
-		)
-	)
 	(global_label "SD_CS"
 		(shape input)
@@
 	(global_label "3V3"
 		(shape input)
-		(at 132.08 38.1 180)
-		(fields_autoplaced yes)
-		(effects
-			(font
-				(size 1.27 1.27)
-			)
-			(justify right)
-		)
-		(property "Intersheetrefs" "${INTERSHEET_REFS}"
-			(at 125.5872 38.1 0)
-			(effects
-				(font
-					(size 1.27 1.27)
-				)
-				(justify right)
-				(hide yes)
-			)
-		)
-	)
-	(global_label "AD0"
-		(shape input)
-		(at 240.03 91.44 180)
+		(at 137.16 46.99 180)
 		(fields_autoplaced yes)
 		(effects
@@
 		)
 		(property "Intersheetrefs" "${INTERSHEET_REFS}"
-			(at 233.4767 91.44 0)
+			(at 130.6672 46.99 0)
 			(effects
 				(font
@@
 			)
 		)
-		(property "Footprint" "Connector_Card:microSD_HC_Hirose_DM3D-SF"
+		(property "Footprint" "Connector_Card:microSD_HC_Hirose_DM3AT-SF-PEJM5"
 			(at -12.7 57.15 0)
 			(effects
@@
 	)
 	(symbol
+		(lib_id "power:GND")
+		(at 140.97 38.1 180)
+		(unit 1)
+		(exclude_from_sim no)
+		(in_bom yes)
+		(on_board yes)
+		(dnp no)
+		(fields_autoplaced yes)
+		(property "Reference" "#PWR05"
+			(at 140.97 31.75 0)
+			(effects
+				(font
+					(size 1.27 1.27)
+				)
+				(hide yes)
+			)
+		)
+		(property "Value" "GND"
+			(at 140.97 33.02 0)
+			(effects
+				(font
+					(size 1.27 1.27)
+				)
+			)
+		)
+		(property "Footprint" ""
+			(at 140.97 38.1 0)
+			(effects
+				(font
+					(size 1.27 1.27)
+				)
+				(hide yes)
+			)
+		)
+		(property "Datasheet" ""
+			(at 140.97 38.1 0)
+			(effects
+				(font
+					(size 1.27 1.27)
+				)
+				(hide yes)
+			)
+		)
+		(property "Description" "Power symbol creates a global label with name \"GND\" , ground"
+			(at 140.97 38.1 0)
+			(effects
+				(font
+					(size 1.27 1.27)
+				)
+				(hide yes)
+			)
+		)
+		(pin "1"
+		)
+		(instances
+			(project ""
+				(path "/04fdbf32-0357-4e6f-8ef5-e0a2d70961b9"
+					(reference "#PWR05")
+					(unit 1)
+				)
+			)
+		)
+	)
+	(symbol
 		(lib_id "Device:R")
 		(at 36.83 93.98 0)
@@
 	(symbol
 		(lib_id "power:GND")
-		(at 140.97 106.68 0)
+		(at 140.97 102.87 0)
 		(unit 1)
 		(exclude_from_sim no)
@@
 		(fields_autoplaced yes)
 		(property "Reference" "#PWR02"
-			(at 140.97 113.03 0)
+			(at 140.97 109.22 0)
 			(effects
 				(font
@@
 		)
 		(property "Value" "GND"
-			(at 140.97 111.76 0)
+			(at 140.97 107.95 0)
 			(effects
 				(font
@@
 		)
 		(property "Footprint" ""
-			(at 140.97 106.68 0)
+			(at 140.97 102.87 0)
 			(effects
 				(font
@@
 		)
 		(property "Datasheet" ""
-			(at 140.97 106.68 0)
+			(at 140.97 102.87 0)
 			(effects
 				(font
@@
 		)
 		(property "Description" "Power symbol creates a global label with name \"GND\" , ground"
-			(at 140.97 106.68 0)
+			(at 140.97 102.87 0)
 			(effects
 				(font
