File: REMOTE IGNITION/Remote ignition system/Remote ignition system.kicad_sch (KiCad schematic)
At the start: 0 parts

Commit message: completed remote ignition circuit
Parts:
- added D1: 1N4007, Diode_THT:D_DO-41_SOD81_P10.16mm_Horizontal, symbol Diode:1N4007
- added J1: RF-reciever, Connector_PinHeader_2.54mm:PinHeader_1x04_P2.54mm_Vertical, symbol Connector:Conn_01x04_Socket
- added J2: BAT_Conn, TerminalBlock_Phoenix:TerminalBlock_Phoenix_MKDS-1,5-2-5.08_1x02_P5.08mm_Horizontal, symbol Connector:Conn_01x02_Socket
- added J3: IGN_BAT, TerminalBlock_Phoenix:TerminalBlock_Phoenix_MKDS-1,5-2-5.08_1x02_P5.08mm_Horizontal, symbol Connector:Conn_01x02_Socket
- added J4: IGN_CONN, TerminalBlock_Phoenix:TerminalBlock_Phoenix_MKDS-1,5-2-5.08_1x02_P5.08mm_Horizontal, symbol Connector:Conn_01x02_Socket
- added K1: Relay_SPDT, Relay_THT:Relay_SPDT_SANYOU_SRD_Series_Form_C, symbol Relay:Relay_SPDT
- added Q1: BC547, Package_TO_SOT_THT:TO-92_Inline, symbol Transistor_BJT:BC547
- added R1: 1kR, Resistor_THT:R_Axial_DIN0207_L6.3mm_D2.5mm_P7.62mm_Horizontal, symbol Device:R
Connections:
- new net: J4.1 (Pin_1), K1.3 (14)
- new net: J3.1 (Pin_1), J4.2 (Pin_2)
- new net: J1.2 (Pin_2), J1.3 (Pin_3), R1.1
- new net: J3.2 (Pin_2), K1.1
- new net: D1.2 (A), K1.2 (12), Q1.3 (E)
- new net DAT: Q1.2 (B), R1.2
- new net GND: J1.1 (Pin_1), J2.2 (Pin_2), Q1.1 (C)
- new net VCC: D1.1 (K), J1.4 (Pin_4), J2.1 (Pin_1), K1.5 (A1)
- no-connect marks 0 -> 1
