File: REMOTE IGNITION/Remote ignition system/Remote ignition system.kicad_pcb (KiCad board)
At the start: 2 copper layers, 57 x 40.5 mm, 8 parts, among them J1 RF-reciever, J2 BAT_Conn, J3 IGN_BAT, J4 IGN_CONN, K1 Relay_SPDT, Q1 BC547

Commit message: Finished remote ignition system
Parts:
- added REF**: MountingHole_2.2mm_M2, MountingHole:MountingHole_2.2mm_M2, F.Cu at (163.5, 124.0)
- added REF**: MountingHole_2.2mm_M2, MountingHole:MountingHole_2.2mm_M2, F.Cu at (111.5, 124.0)
- added REF**: MountingHole_2.2mm_M2, MountingHole:MountingHole_2.2mm_M2, F.Cu at (163.5, 88.5)
- added REF**: MountingHole_2.2mm_M2, MountingHole:MountingHole_2.2mm_M2, F.Cu at (111.5, 88.5)
- moved J4 3.57 mm to (152.4, 120.7)
- moved J3 3.50 mm to (157.5, 92.3)
- moved J2 2.00 mm to (124.0, 92.5)
Routing:
- net Net-(J3-Pin_2): track 28.7 -> 25.2 mm
- net Net-(J3-Pin_1): track 27.6 -> 30.4 mm
- net Net-(J4-Pin_1): track 11.3 -> 9.68 mm
- net VCC: track 42.7 -> 41.6 mm
- net GND: track 29.1 -> 29.8 mm
